File: output_mixer.kicad_pcb (KiCad board)
At the start: 2 copper layers, 40 x 99 mm, 114 parts, among them J1 IN1, J2 IN2, J3 IN1, J4 IN2, J5 Headphones, J6 Line out, Q2 BD139, Q3 BD140, Q4 BD139, Q5 BD140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

Commit message: Design done and sent to production
Parts:
- J5, J6: footprint Connector_Audio:Jack_3.5mm_QingPu_WQP-PJ398SM_Vertical_CircularHoles_Stereo -> AudioJacks:Jack_3.5mm_Stereo_Unbranded
- moved R33 226.8 mm to (275.5, 92.0), turned to 90 degrees
- moved R28 212.8 mm to (260.5, 103.0), turned to 90 degrees
- moved R29 210.6 mm to (258.5, 103.0), turned to -90 degrees
- moved R30 207.1 mm to (255.5, 99.0)
- moved R39 205.1 mm to (256.0, 103.0), turned to -90 degrees
- moved R58 196.6 mm to (253.5, 103.0), turned to -90 degrees
- moved R59 194.1 mm to (251.5, 99.0), turned to 180 degrees
- moved D18 179.6 mm to (248.0, 99.5), turned to -90 degrees
- moved D17 179.4 mm to (248.0, 83.5), turned to 90 degrees
- moved C17 177.2 mm to (273.5, 92.0), turned to -90 degrees
- moved TP5 172.9 mm to (265.6, 16.8)
- moved D11 170.0 mm to (261.0, 107.5), turned to -90 degrees
- moved C4 169.8 mm to (248.0, 109.0), turned to 180 degrees
- moved D13 166.9 mm to (267.0, 73.0)
- moved D12 166.9 mm to (258.5, 107.5), turned to 90 degrees
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Routing:
- net -12V: track 0.00 -> 240.1 mm, vias 0 -> 7
- net +12V: track 0.00 -> 232.9 mm, vias 0 -> 10
- net GND: track 0.00 -> 218.2 mm, vias 0 -> 15
- net Net-(U3B--): track 0.00 -> 103.7 mm
- net Net-(U3A--): track 0.00 -> 87.7 mm, vias 0 -> 7
- net Net-(U2B--): track 0.00 -> 74.0 mm, vias 0 -> 4
- net Net-(R13-Pad1): track 0.00 -> 64.1 mm, vias 0 -> 4
- net Net-(C16-Pad2): track 0.00 -> 58.1 mm, vias 0 -> 1
- net Net-(R46-Pad1): track 0.00 -> 55.4 mm, vias 0 -> 2
- net Net-(D1-K): track 0.00 -> 55.0 mm
- net Net-(D7-K): track 0.00 -> 51.5 mm, vias 0 -> 4
- net Net-(D3-K): track 0.00 -> 46.8 mm, vias 0 -> 1
- net Net-(C17-Pad2): track 0.00 -> 45.2 mm, vias 0 -> 1
- net Net-(D5-K): track 0.00 -> 42.9 mm
- net Net-(D10-K): track 0.00 -> 42.0 mm, vias 0 -> 2
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- added copper zone on B.Cu, net GND
- added copper zone on F.Cu, net GND
Other:
- outline, holes or cut-outs redrawn
- board text added: "HEADPHONE OUT"
- board text added: "IN 1"
- board text added: "IN 2"
- board text added: "IN 3"
- board text added: "IN 4"
- board text added: "JLCJLCJLCJLC"
- board text added: "LINE OUT"
- board text added: "LVL 1"
- board text added: "LVL 2"
- board text added: "LVL 3"
- board text added: "LVL 4"
- board text added: "Output mixer design by mohoyt"
- board text added: "PAN 1"
- board text added: "PAN 2"
- board text added: "PAN 3"
- board text added: "PAN 4"

Commit message: v1 issues fixed (opposite panning and 47R resistor footprint size)
Parts:
- R26, R38: footprint Resistor_THT:R_Axial_DIN0207_L6.3mm_D2.5mm_P7.62mm_Horizontal -> Resistor_THT:R_Axial_DIN0309_L9.0mm_D3.2mm_P12.70mm_Horizontal
- moved R26 9.24 mm to (275.2, 95.5)
- moved R36 3.20 mm to (264.5, 95.5)
- moved R37 2.80 mm to (272.5, 98.9)
- moved R38 0.70 mm to (263.0, 111.9)
- moved R2 0.29 mm to (253.3, 112.0)
Connections:
- R23 pad 1: Net-(R23-Pad1) -> Net-(R21-Pad1)
- R23 pad 3: Net-(R21-Pad1) -> Net-(R23-Pad3)
- R27 pad 1: Net-(R23-Pad1) -> Net-(R23-Pad3)
- R31 pad 2: Net-(R23-Pad1) -> Net-(R23-Pad3)
- R49 pad 1: Net-(R48-Pad1) -> Net-(R47-Pad1)
- R49 pad 3: Net-(R47-Pad1) -> Net-(R48-Pad1)
- R52 pad 1: Net-(R15-Pad1) -> Net-(R14-Pad1)
- R52 pad 3: Net-(R14-Pad1) -> Net-(R15-Pad1)
- R53 pad 1: Net-(R17-Pad1) -> Net-(R16-Pad1)
- R53 pad 3: Net-(R16-Pad1) -> Net-(R17-Pad1)
Routing:
- net Net-(R23-Pad1): track 25.1 -> 0.00 mm, vias 1 -> 0
- net Net-(R23-Pad3): track 0.00 -> 24.7 mm, vias 0 -> 3
- net Net-(R21-Pad1): track 18.5 -> 24.7 mm
- net Net-(R14-Pad1): track 20.1 -> 25.8 mm, vias 2 -> 3
- net Net-(R17-Pad1): track 26.6 -> 21.5 mm
- net Net-(R47-Pad1): track 31.1 -> 36.1 mm
- net Net-(R48-Pad1): track 31.9 -> 26.9 mm
- net Net-(R16-Pad1): track 29.5 -> 32.8 mm, vias 3 -> 4
- net Net-(J5-PadR): track 7.54 -> 9.05 mm
- net Net-(Q4-E): track 13.3 -> 14.5 mm
- net Net-(C16-Pad2): track 58.1 -> 59.1 mm
- net -12V: track 240.1 -> 239.3 mm
- net Net-(J5-PadT): track 15.5 -> 16.1 mm
