File: output_mixer.kicad_sch (KiCad schematic)
At the start: 114 parts, among them J1 IN1, J2 IN2, J3 IN1, J4 IN2, J5 Headphones, J6 Line out, Q2 BD139, Q3 BD140, Q4 BD139, Q5 BD140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

Commit message: v1 issues fixed (opposite panning and 47R resistor footprint size)
Parts:
- R26, R38: footprint Resistor_THT:R_Axial_DIN0207_L6.3mm_D2.5mm_P7.62mm_Horizontal -> Resistor_THT:R_Axial_DIN0309_L9.0mm_D3.2mm_P12.70mm_Horizontal
Connections:
- net at R47.1, R50.2: now also R49.1; no longer R49.3
- net at R17.1, R57.2: now also R53.3; no longer R53.1
- net at R14.1, R54.2: now also R52.1; no longer R52.3
- net at R16.1, R56.2: now also R53.1; no longer R53.3
- net at R27.1, R31.2: now also R23.3; no longer R23.1
- net at R15.1, R55.2: now also R52.3; no longer R52.1
- net at R48.1, R51.2: now also R49.3; no longer R49.1
- net at R21.1, R22.2: now also R23.1; no longer R23.3
Changed lines of the file:
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@@
       (effects (font (size 1.27 1.27)))
     )
-    (property "Footprint" "Resistor_THT:R_Axial_DIN0207_L6.3mm_D2.5mm_P7.62mm_Horizontal" (at 240.03 100.838 90)
+    (property "Footprint" "Resistor_THT:R_Axial_DIN0309_L9.0mm_D3.2mm_P12.70mm_Horizontal" (at 240.03 100.838 90)
       (effects (font (size 1.27 1.27)) hide)
     )
@@
     )
   )
-  (symbol (lib_id "Device:R_Potentiometer") (at 129.54 149.86 0) (mirror x) (unit 1)
+  (symbol (lib_id "Device:R_Potentiometer") (at 129.54 149.86 0) (unit 1)
     (in_bom yes) (on_board yes) (dnp no)
-    (property "Reference" "R52" (at 127 150.495 0)
+    (property "Reference" "R52" (at 127 149.225 0)
       (effects (font (size 1.27 1.27)) (justify right))
     )
-    (property "Value" "B10k" (at 127 147.955 0)
+    (property "Value" "B10k" (at 127 151.765 0)
       (effects (font (size 1.27 1.27)) (justify right))
     )
@@
     )
   )
-  (symbol (lib_id "Device:R_Potentiometer") (at 128.27 115.57 0) (mirror x) (unit 1)
+  (symbol (lib_id "Device:R_Potentiometer") (at 128.27 115.57 0) (unit 1)
     (in_bom yes) (on_board yes) (dnp no)
-    (property "Reference" "R49" (at 125.73 116.205 0)
+    (property "Reference" "R49" (at 125.73 114.935 0)
       (effects (font (size 1.27 1.27)) (justify right))
     )
-    (property "Value" "B10k" (at 125.73 113.665 0)
+    (property "Value" "B10k" (at 125.73 117.475 0)
       (effects (font (size 1.27 1.27)) (justify right))
     )
@@
       (effects (font (size 1.27 1.27)))
     )
-    (property "Footprint" "Resistor_THT:R_Axial_DIN0207_L6.3mm_D2.5mm_P7.62mm_Horizontal" (at 242.57 191.008 90)
+    (property "Footprint" "Resistor_THT:R_Axial_DIN0309_L9.0mm_D3.2mm_P12.70mm_Horizontal" (at 242.57 191.008 90)
       (effects (font (size 1.27 1.27)) hide)
     )
@@
     )
   )
-  (symbol (lib_id "Device:R_Potentiometer") (at 129.54 182.88 0) (mirror x) (unit 1)
+  (symbol (lib_id "Device:R_Potentiometer") (at 129.54 182.88 0) (unit 1)
     (in_bom yes) (on_board yes) (dnp no)
-    (property "Reference" "R53" (at 127 183.515 0)
+    (property "Reference" "R53" (at 127 182.245 0)
       (effects (font (size 1.27 1.27)) (justify right))
     )
-    (property "Value" "B10k" (at 127 180.975 0)
+    (property "Value" "B10k" (at 127 184.785 0)
       (effects (font (size 1.27 1.27)) (justify right))
     )
@@
     )
   )
-  (symbol (lib_id "Device:R_Potentiometer") (at 128.27 82.55 0) (mirror x) (unit 1)
+  (symbol (lib_id "Device:R_Potentiometer") (at 128.27 82.55 0) (unit 1)
     (in_bom yes) (on_board yes) (dnp no)
-    (property "Reference" "R23" (at 125.73 83.185 0)
+    (property "Reference" "R23" (at 125.73 81.915 0)
       (effects (font (size 1.27 1.27)) (justify right))
     )
-    (property "Value" "B10k" (at 125.73 80.645 0)
+    (property "Value" "B10k" (at 125.73 84.455 0)
       (effects (font (size 1.27 1.27)) (justify right))
     )
